File: pnp55te.kicad_pcb (KiCad board)
At the start: 2 copper layers, 154 x 109 mm, 68 parts, among them P1 1123038-2, U1 VNLD5090, U2 VNLD5090, U3 molex_48pin_MRE, U4 ITEAD_HC-05

Commit message: progress
Other:
- outline, holes or cut-outs redrawn
- board text added: "Vertical clearance: (including PCB material) 8.3mm total on sides 10.3 (2mm extra) in the middle"
Changed lines of the file:
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@@
   (general
     (thickness 1.6)
-    (drawings 25)
+    (drawings 26)
     (tracks 0)
     (zones 0)
@@
     )
   )
+  (gr_text "Vertical clearance:\n(including PCB material)\n8.3mm total on sides\n10.3 (2mm extra) in the middle" (at -28.6 -18.8) (layer Cmts.User)
+    (effects (font (size 4 4) (thickness 0.15)))
+  )
   (gr_line (start 124 5.7) (end 30 5.7) (layer Edge.Cuts) (width 0.2))
   (gr_line (start 124 21.9) (end 124 5.7) (layer Edge.Cuts) (width 0.2))
   (gr_line (start 30 21.9) (end 124 21.9) (layer Edge.Cuts) (width 0.2))
   (gr_line (start 30 5.7) (end 30 21.9) (layer Edge.Cuts) (width 0.2))
-  (gr_circle (center 131.5 10) (end 134 10) (layer Edge.Cuts) (width 0.2))
+  (gr_circle (center 131.5 10) (end 134.3 10) (layer Edge.Cuts) (width 0.2))
   (gr_line (start 0 94) (end 15 109) (layer Edge.Cuts) (width 0.1))
   (gr_line (start 139 109) (end 154 94) (layer Edge.Cuts) (width 0.1))
@@
     (effects (font (size 1.5 1.5) (thickness 0.3)))
   )
-  (gr_circle (center 32 99) (end 34.5 99) (layer Edge.Cuts) (width 0.2))
-  (gr_circle (center 122 99) (end 124.5 99) (layer Edge.Cuts) (width 0.2))
-  (gr_circle (center 149.5 54) (end 152 54) (layer Edge.Cuts) (width 0.2))
-  (gr_circle (center 22.5 10) (end 25 10) (layer Edge.Cuts) (width 0.2))
-  (gr_circle (center 4.5 54) (end 7 54) (layer Edge.Cuts) (width 0.2))
+  (gr_circle (center 32 99) (end 34.8 99) (layer Edge.Cuts) (width 0.2))
+  (gr_circle (center 122 99) (end 124.8 99) (layer Edge.Cuts) (width 0.2))
+  (gr_circle (center 149.5 54) (end 152.3 54) (layer Edge.Cuts) (width 0.2))
+  (gr_circle (center 22.5 10) (end 25.3 10) (layer Edge.Cuts) (width 0.2))
+  (gr_circle (center 4.5 54) (end 7.3 54) (layer Edge.Cuts) (width 0.2))
   (gr_line (start 15 0) (end 139 0) (layer Edge.Cuts) (width 0.1))
   (gr_line (start 154 15) (end 154 94) (layer Edge.Cuts) (width 0.1))

Commit message: Update schematic and PCB with bew symbol and footprint
Parts:
- removed C1, C2, C3, C4: 6.8n, Capacitor_SMD:C_0603_1608Metric
- removed C5: 0.1u, Capacitor_SMD:C_0805_2012Metric
- removed C6: 1u, Capacitor_SMD:C_0805_2012Metric
- removed D1, D2, D5, D6: D_Schottky, Diode_SMD:D_SMF
- removed D3, D4, D7, D8: LED, LED_SMD:LED_0603_1608Metric
- removed P1: 1123038-2, rusefi_pretty:1123038-2
- removed R1, R11, R12, R2, R5, R6, R7, R8: 1k, Resistor_SMD:R_0603_1608Metric
- removed R10, R3, R4, R9: 10k, Resistor_SMD:R_0603_1608Metric
- removed U1, U2: VNLD5090, Package_SO:SO-8_3.9x4.9mm_P1.27mm
- removed U3: molex_48pin_MRE, rusEFI_Modules:Molex_48_MRE_with-extras
- removed U4: ITEAD_HC-05, rusEFI_Modules:ITEAD_HC-05
- removed W1, W10, W11, W12, W13, W14, W15, W16, W17, W18, W19, W2, W20, W21, W22, W23, W24, W25, W26, W27, W28, W29, W3, W30, W31, W32, W33, W34, W35, W36, W37, W4, W5, W6, W7, W8, W9: TestPoint_2Pole, rusEFI_Modules:SM0805_jumper
- added U?1: molex_48pin_MRE, rusEFI_Modules:Molex_48_MRE_with-extras, F.Cu at (75.6, 123.8)
- added X1: 55pin_january_5.1, hw_55_te:55pin_january_5.1, F.Cu at (96.5, 43.8)
Other:
- outline, holes or cut-outs redrawn

Commit message: Use correct connector name
Parts:
- X1: footprint hw_55_te:55pin_january_5.1 -> hw_55_te:TE_963063-2
