File: motronic-wire-adapter.kicad_pcb (KiCad board)
At the start: 2 copper layers, 157.5 x 48.5 mm, 10 parts, among them P1 MOTRONIC, P2 CONN_19, P3 CONN_18, P4 CONN_18, P5 CONN_1, P6 CONN_1

Commit message: Use pattern from kicad-libraries
Parts:
- P1: footprint hw_55_te:55pin_china_bosch_motronic -> rusEFI_Modules:55pin_china_bosch_motronic
Changed lines of the file:
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@@
     (add_net N-000009)
   )
-  (module hw_55_te:55pin_china_bosch_motronic (layer F.Cu)
+  (module rusEFI_Modules:55pin_china_bosch_motronic (layer F.Cu)
     (at 220 168.5 180)
     (fp_text reference P1 (at 0 27.5) (layer F.SilkS) hide
